File: main.brd (EAGLE design)
At the start: 400 x 300 mm, 474 parts, among them J100 DCJ0202, Q200 NMOS, Q201 PMOS, Q300 PMOS, Q400 PMOS, U100 NE555N, U1000 74LS173N, U1001 74LS173N, U1002 74LS245N, U1003 74LS173N, U1004 74LS173N, U1005 74LS245N, U101 NE555N, U102 NE555N, U103 74LS04N, U104 74LS08N, U105 74LS32N, U1100 74LS173N, U1101 74LS173N, U1102 74LS161N, U1106 74HCT154DW, U1107 74HCT154DW, U1108 74LS04N, U1109 74LS04N, U200 HM62256, U201 74LS173N, U202 74LS173N, U203 74LS173N, U204 74LS173N, U205 74LS157N, U206 74LS157N, U207 74LS157N, U208 74LS157N, U209 74HCT595D, U210 74HCT595D, U211 74HCT595D, U212 74LS245N, U213 74LS245N, U214 74LS00N, U215 74LS173N, U216 74LS173N, U217 74LS173N, U218 74LS173N, U219 74LS245N, U220 74LS245N, U300 74LS299N, U301 74LS245N, U302 74LS08N, U303 74LS00N, U304 74LS245N, U400 74LS00N, U401 74LS245N, U500 74LS161N, U501 74LS161N, U502 74LS161N, U503 74LS161N, U504 74LS245N, U505 74LS245N, U600 74LS173N, U601 74LS173N, U602 74LS173N, U603 74LS173N, U604 74LS245N, U700 74LS283N, U701 74LS283N, U702 74LS245N, U703 74LS86N, U704 74LS86N, U705 74LS85N, U706 74LS85N, U707 74LS173N, U708 74LS125N, U800 74LS04N, U801 74LS04N, U802 74LS08N, U803 74LS08N, U804 74LS32N, U805 74LS32N, U806 74LS86N, U807 74LS86N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

Commit message: Z register mostly done.
Parts:
- moved U219 468.2 mm to (212.1, 72.4), turned to 180 degrees
- moved LED232 436.0 mm to (201.9, 80.4)
- moved U220 432.3 mm to (142.2, 72.4), turned to 180 degrees
- moved LED231 430.1 mm to (207.0, 80.4)
- moved LED230 424.1 mm to (212.1, 80.4)
- moved LED229 418.2 mm to (217.2, 80.4)
- moved RN206 417.6 mm to (242.6, 80.4), flipped to the bottom, turned to 90 degrees
- moved LED228 412.3 mm to (222.2, 80.4)
- moved LED227 406.5 mm to (227.3, 80.4)
- moved LED226 400.6 mm to (232.4, 80.4)
- moved LED225 394.7 mm to (237.5, 80.4)
- moved C215 380.7 mm to (125.7, 83.8)
- moved C216 380.7 mm to (120.7, 83.8)
- moved C217 380.7 mm to (115.6, 83.8)
- moved C218 380.7 mm to (110.5, 83.8)
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Connections:
- net LED225_GND: now also RN206.4; no longer RN206.1
- net LED226_GND: now also RN206.3; no longer RN206.2
- net LED227_GND: now also RN206.2; no longer RN206.3
- net LED228_GND: now also RN206.1; no longer RN206.4
Routing:
- net GND: track 2488.3 -> 2643.8 mm
- net MAINBUS_0: track 721.4 -> 848.4 mm, vias 4 -> 7
- net MAINBUS_1: track 658.5 -> 784.5 mm, vias 6 -> 9
- net MAINBUS_2: track 648.3 -> 773.4 mm, vias 6 -> 9
- net MAINBUS_3: track 607.3 -> 731.2 mm, vias 4 -> 7
- net MAINBUS_4: track 586.7 -> 698.9 mm, vias 4 -> 7
- net MAINBUS_5: track 580.9 -> 692.0 mm, vias 4 -> 7
- net MAINBUS_6: track 570.2 -> 679.8 mm, vias 4 -> 7
- net MAINBUS_7: track 546.3 -> 652.8 mm
- net CLK: track 657.9 -> 757.8 mm, vias 19 -> 23
- net REG_Z_11: track 0.00 -> 44.6 mm, vias 0 -> 1
- net REG_Z_3: track 0.00 -> 44.6 mm, vias 0 -> 1
- net REG_Z_2: track 0.00 -> 44.2 mm, vias 0 -> 1
- net REG_Z_10: track 0.00 -> 44.2 mm, vias 0 -> 1
- net REG_Z_1: track 0.00 -> 43.8 mm, vias 0 -> 1
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
Commit message: Finished Z, V and F registers.
Parts:
- moved LED1000 827.6 mm to (97.8, 139.3)
- moved LED1001 812.8 mm to (102.9, 139.3)
- moved U1002 812.2 mm to (108.0, 147.6)
- moved U1000 808.9 mm to (132.1, 147.6)
- moved LED1002 798.1 mm to (108.0, 139.3)
- moved LED1003 783.6 mm to (113.0, 139.3)
- moved U1001 773.4 mm to (153.7, 147.6)
- moved LED1004 769.1 mm to (118.1, 139.3)
- moved LED1008 765.7 mm to (167.6, 139.3)
- moved C1000 764.6 mm to (121.3, 152.0), flipped to the bottom, turned to 270 degrees
- moved C1002 759.6 mm to (121.3, 143.3), flipped to the bottom, turned to 270 degrees
- moved LED1005 754.9 mm to (123.2, 139.3)
- moved RN1000 751.8 mm to (138.4, 139.3), flipped to the bottom, turned to 90 degrees
- moved LED1009 751.3 mm to (172.7, 139.3)
- moved LED1006 740.7 mm to (128.3, 139.3)
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Connections:
- net LED1004_GND: now also RN1000.8; no longer RN1000.5
- net LED1005_GND: now also RN1000.7; no longer RN1000.6
- net LED1006_GND: now also RN1000.6; no longer RN1000.7
- net LED1007_GND: now also RN1000.5; no longer RN1000.8
- net LED1012_GND: now also RN1001.8; no longer RN1001.5
- net LED1013_GND: now also RN1001.7; no longer RN1001.6
- net LED1014_GND: now also RN1001.6; no longer RN1001.7
- net LED1015_GND: now also RN1001.5; no longer RN1001.8
- net LED237_GND: now also RN207.8; no longer RN207.5
- net LED238_GND: now also RN207.7; no longer RN207.6
- net LED239_GND: now also RN207.6; no longer RN207.7
- net LED240_GND: now also RN207.5; no longer RN207.8
Routing:
- net VCC: track 1921.4 -> 2280.0 mm, vias 34 -> 36
- net GND: track 2643.8 -> 2915.2 mm, vias 34 -> 38
- net RST: track 205.3 -> 405.2 mm, vias 3 -> 11
- net MAINBUS_0: track 848.4 -> 970.3 mm, vias 7 -> 10
- net MAINBUS_1: track 784.5 -> 905.5 mm, vias 9 -> 12
- net MAINBUS_2: track 773.4 -> 893.4 mm, vias 9 -> 12
- net MAINBUS_3: track 731.2 -> 850.0 mm, vias 7 -> 10
- net MAINBUS_4: track 698.9 -> 806.0 mm, vias 7 -> 10
- net MAINBUS_5: track 692.0 -> 798.0 mm, vias 7 -> 10
- net MAINBUS_6: track 679.8 -> 784.3 mm, vias 7 -> 10
- net MAINBUS_7: track 652.8 -> 754.2 mm
- net CLK: track 757.8 -> 857.7 mm, vias 23 -> 27
- net REG_F_0: track 0.00 -> 60.0 mm
- net REG_V_0: track 0.00 -> 60.0 mm
- net REG_V_1: track 0.00 -> 58.7 mm, vias 0 -> 1
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
Commit message: Cleanup and routing of all non-CTRL signals.
Parts:
- moved LED308 414.6 mm to (110.4, 296.7), turned to 180 degrees
- moved LED309 407.5 mm to (115.4, 296.7), turned to 180 degrees
- moved LED310 401.0 mm to (120.5, 296.7), turned to 180 degrees
- moved LED311 395.0 mm to (125.6, 296.7), turned to 180 degrees
- moved LED312 389.7 mm to (130.7, 296.7), turned to 180 degrees
- moved LED313 385.0 mm to (135.8, 296.7), turned to 180 degrees
- moved RN302 384.1 mm to (126.9, 292.0), flipped to the bottom, turned to 180 degrees
- moved LED314 381.0 mm to (140.8, 296.7), turned to 180 degrees
- moved LED315 377.7 mm to (145.9, 296.7), turned to 180 degrees
- moved J100 25.9 mm to (66.0, 289.6), turned to 180 degrees
- moved LED1006 16.8 mm to (115.6, 150.2)
- moved LED1010 16.8 mm to (165.1, 150.2)
- moved LED1012 16.8 mm to (175.3, 150.2)
- moved LED1014 16.8 mm to (185.4, 150.2)
- moved LED226 16.8 mm to (185.4, 178.9)
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Routing:
- net RST: track 405.2 -> 638.2 mm
- net !RST: track 119.9 -> 230.8 mm, vias 0 -> 1
- net MAINBUS_4: track 806.0 -> 902.2 mm
- net MAINBUS_6: track 784.3 -> 880.4 mm
- net MAINBUS_7: track 754.2 -> 848.7 mm
- net MAINBUS_5: track 798.0 -> 890.5 mm
- net MAINBUS_3: track 850.0 -> 932.5 mm
- net MAINBUS_2: track 893.4 -> 973.2 mm
- net MAINBUS_1: track 905.5 -> 983.2 mm
- net MAINBUS_0: track 970.3 -> 1044.5 mm
- net CLK: track 857.7 -> 922.2 mm
- net MEM_MANMODE: track 138.0 -> 176.7 mm, vias 2 -> 3
- net VCC: track 2280.0 -> 2312.8 mm
- net LED315_GND: track 0.00 -> 18.3 mm
- net LED308_GND: track 0.00 -> 18.3 mm
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
Commit message: Routing and layout done.
Parts:
- removed C1109: 0.1µF, rcl:C0805K
- removed U1109: 74LS04N, 74xx-us:DIL14
- added C709: 0.1µF, rcl:C0805K
- added J400: 90152-12, 8BitCpuParts:90152-12
- added LED401: (no value), led:CHIP-LED0805
- added Q401, Q402: NMOS, ExtraParts:SOT23
- added R1103: 330Ω?, resistor:R0805
- added R403: 10kΩ, resistor:R0805
- added R404: 1kΩ, resistor:R0805
- added S402: NK236H, 8BitCpuParts:NK236*H
- added U709: 74LS153N, 74xx-us:DIL16
- moved LED1112 874.7 mm to (294.6, 45.5)
- moved LED1111 855.8 mm to (289.6, 45.5)
- moved LED1148 850.8 mm to (291.7, 69.1)
- moved LED1164 848.1 mm to (303.8, 66.5), turned to 180 degrees
- moved LED1158 845.3 mm to (303.8, 97.0), turned to 180 degrees
- moved LED1110 845.2 mm to (255.3, 42.4)
- moved LED1102 840.1 mm to (247.7, 37.3)
- moved LED1147 838.7 mm to (291.7, 74.2)
- moved LED1163 836.2 mm to (303.8, 71.6), turned to 180 degrees
- moved LED1118 835.0 mm to (281.9, 45.5)
- moved LED1130 832.3 mm to (286.9, 84.3), turned to 180 degrees
- moved LED1101 829.5 mm to (242.6, 37.3)
- moved LED1146 826.7 mm to (291.7, 79.2)
- moved LED1162 824.3 mm to (303.8, 76.7), turned to 180 degrees
- moved LED1117 824.2 mm to (276.9, 45.5)
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Connections:
- net CMP_= renamed CMP_EQ_INT
- removed net CMP_<: U706.7, U707.14
- removed net CMP_>: U706.5, U707.12
- removed net CTRL_15: LED1164.A, XU1105.19
- removed net OUT_15: U1108.8
- new net CMP_GT_INT: U707.12, U709.9
- new net CMP_GT_PRE: U706.5, U709.10, U709.11, U709.12, U709.3
- new net CMP_LT_INT: U707.14, U709.7
- new net CMP_LT_PRE: U706.7, U709.13, U709.4, U709.5, U709.6
- new net CPTC: LED1153.A, U709.2, XU1104.16
- new net INPUT_GND: Q401.3, S400.B1, S400.B2, S400.B3, S400.B4, S400.B5, S400.B6, S400.B7, S400.B8
- new net INPUT_GND_INT: Q401.2, Q402.3
- new net INPUT_LOCK_ARDUINO: A200.8, Q401.1, R403.1
- new net INPUT_LOCK_EXT: LED401.C, Q402.1, S402.C
- new net LED401_VCC: LED401.A, R404.2
- net !CLK: now also U800.12
- net !CMP: now also U800.2; no longer U1109.2
- net !FE: now also U1108.10; no longer U1109.4
- net !NO: now also A200.26, J400.3
- net !OUT_15: no longer U1108.9
- net !RM: now also U1108.6; no longer U1109.6
- net !RMSB: now also U1108.8; no longer U1109.8
- net !RO: now also U1108.13; no longer U1108.5
- net BITWISE_XOR_7: now also U709.14
- net CLK: now also U800.13
- net CMP: now also U800.1; no longer U1109.1
- net FE: now also LED1154.A, U1108.11, XU1104.17; no longer LED1153.A, U1109.3, XU1104.16
- net GND: now also C709.2, J400.1, Q402.2, R1103.2, S402.2, U709.1, U709.15, U709.8; no longer C1109.2, S400.B1, S400.B2, S400.B3, S400.B4, S400.B5, S400.B6, S400.B7, S400.B8, U1109.7
- net HLT: now also LED1155.A, XU1104.18; no longer LED1154.A, XU1104.17
- net INPUT_0: now also A200.27, J400.5
- net INPUT_1: now also A200.28, J400.7
- net INPUT_2: now also A200.29, J400.9
- net INPUT_3: now also A200.30, J400.11
- net INPUT_4: now also A200.4, J400.6
- net INPUT_5: now also A200.5, J400.8
- net INPUT_6: now also A200.6, J400.10
- net INPUT_7: now also A200.7, J400.12
- net LED1107_GND: now also R1100.1; no longer RN1100.8
- net LED1108_GND: now also R1101.1; no longer R1100.1
- net LED1109_GND: now also R1102.1; no longer R1101.1
- net LED1110_GND: now also R1103.1; no longer R1102.1
- net LED1111_GND: now also RN1101.8; no longer RN1101.1
- net LED1112_GND: now also RN1101.7; no longer RN1101.2
- net LED1113_GND: now also RN1101.6; no longer RN1101.3
- net LED1114_GND: now also RN1101.5; no longer RN1101.4
- net LED1115_GND: now also RN1101.4; no longer RN1101.5
- net LED1116_GND: now also RN1101.3; no longer RN1101.6
- net LED1117_GND: now also RN1101.2; no longer RN1101.7
- net LED1118_GND: now also RN1101.1; no longer RN1101.8
- net LED1134_VCC: now also RN1104.7; no longer RN1104.2
- net LED1135_VCC: now also RN1104.6; no longer RN1104.3
- net LED1136_VCC: now also RN1104.5; no longer RN1104.4
- net LED1137_VCC: now also RN1104.4; no longer RN1104.5
- net LED1138_VCC: now also RN1104.3; no longer RN1104.6
- net LED1139_VCC: now also RN1104.2; no longer RN1104.7
- net LED1140_VCC: now also RN1104.1; no longer RN1104.8
- net LED1141_VCC: now also RN1105.8; no longer RN1105.1
- net LED1142_VCC: now also RN1105.7; no longer RN1105.2
- net LED1143_VCC: now also RN1105.6; no longer RN1105.3
- net LED1144_VCC: now also RN1105.5; no longer RN1105.4
- net LED1145_VCC: now also RN1105.4; no longer RN1105.5
- net LED1146_VCC: now also RN1105.3; no longer RN1105.6
- net LED1147_VCC: now also RN1105.2; no longer RN1105.7
- net LED1148_VCC: now also RN1105.1; no longer RN1105.8
- net LED1149_GND: now also RN1106.8; no longer RN1106.1
- net LED1150_GND: now also RN1106.7; no longer RN1106.2
- net LED1151_GND: now also RN1106.6; no longer RN1106.3
- net LED1152_GND: now also RN1106.5; no longer RN1106.4
- net LED1153_GND: now also RN1106.4; no longer RN1106.5
- net LED1154_GND: now also RN1106.3; no longer RN1106.6
- net LED1155_GND: now also RN1106.2; no longer RN1106.7
- net LED1156_GND: now also RN1106.1; no longer RN1106.8
- net LED1157_GND: now also RN1107.8; no longer RN1107.1
- net LED1158_GND: now also RN1107.7; no longer RN1107.2
- net LED1159_GND: now also RN1107.6; no longer RN1107.3
- net LED1160_GND: now also RN1107.5; no longer RN1107.4
- net LED1161_GND: now also RN1107.4; no longer RN1107.5
- net LED1162_GND: now also RN1107.3; no longer RN1107.6
- net LED1163_GND: now also RN1107.2; no longer RN1107.7
- net LED1164_GND: now also RN1107.1; no longer RN1107.8
- net NO_RESET_PULSE: now also A200.25, J400.4
- net RM: now also LED1156.A, U1108.5, XU1104.19; no longer LED1155.A, U1109.5, XU1104.18
- net RMSB: now also LED1157.A, U1108.9, XU1105.11; no longer LED1156.A, U1109.9, XU1104.19
- net RO: now also U1108.12; no longer U1108.6
- net SM0: now also LED1158.A, XU1105.12; no longer LED1157.A, XU1105.11
- net SM1: now also LED1159.A, XU1105.13; no longer LED1158.A, XU1105.12
- net SRO: now also LED1160.A, XU1105.15; no longer LED1159.A, XU1105.13
- net SUB: now also LED1161.A, XU1105.16; no longer LED1160.A, XU1105.15
- net T0: now also LED1162.A, XU1105.17; no longer LED1161.A, XU1105.16
- net T1: now also LED1163.A, XU1105.18; no longer LED1162.A, XU1105.17
- net VCC: now also C709.1, J400.2, R403.2, R404.1, S402.1, U709.16; no longer C1109.1, U1109.14
- net XR: now also LED1164.A, XU1105.19; no longer LED1163.A, XU1105.18
Routing:
- net GND: track 2897.1 -> 3707.2 mm, vias 38 -> 57
- net !NO: track 34.0 -> 686.6 mm, vias 0 -> 7
- net VCC: track 2312.8 -> 2833.8 mm, vias 36 -> 47
- net HLT: track 0.00 -> 470.9 mm, vias 0 -> 5
- net SRO: track 12.3 -> 469.9 mm, vias 0 -> 5
- net SM1: track 98.0 -> 553.4 mm, vias 1 -> 6
- net SM0: track 102.2 -> 548.2 mm, vias 1 -> 6
- net !SO: track 0.00 -> 412.5 mm, vias 0 -> 4
- net XR: track 0.00 -> 399.5 mm, vias 0 -> 3
- net FE: track 0.00 -> 393.1 mm, vias 0 -> 4
- net !RI: track 0.00 -> 387.3 mm, vias 0 -> 4
- net !RO: track 0.00 -> 383.1 mm, vias 0 -> 4
- net !XI: track 0.00 -> 378.5 mm, vias 0 -> 4
- net RMSB: track 0.00 -> 378.5 mm, vias 0 -> 4
- net RM: track 0.00 -> 369.0 mm, vias 0 -> 4
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Other:
- board size 400 x 300 mm -> 314.5 x 159.5 mm

Commit message: Revised external input, progress on silkscreen.
Parts:
- removed LED401: (no value), led:CHIP-LED0805
- removed S402: NK236H, 8BitCpuParts:NK236*H
- J400: value 90152-12 -> 90152-14; device 8BitCpuParts:90152-12 -> 8BitCpuParts:90152-14
- R404: value 1kΩ -> 10kΩ
- moved R404 116.7 mm to (120.6, 53.8), flipped to the bottom, turned to 270 degrees
- moved J400 6.10 mm to (4.80, 27.4)
- moved C501 0.25 mm to (195.6, 132.5)
- moved C503 0.25 mm to (198.5, 146.1)
- moved C504 0.25 mm to (152.1, 134.4)
- moved C809 0.25 mm to (232.9, 132.1)
- moved C811 0.25 mm to (255.8, 132.1)
- moved C812 0.25 mm to (242.8, 147.2)
- moved LED101 0.25 mm to (2.92, 132.1)
- moved LED1120 0.25 mm to (286.9, 135.4)
- moved LED1135 0.25 mm to (291.7, 135.4)
- moved LED1149 0.25 mm to (303.8, 143.0)
- moved LED1151 0.25 mm to (303.8, 132.8)
- moved Q300 0.25 mm to (143.5, 134.7)
- moved R100 0.25 mm to (9.91, 156.2)
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Connections:
- removed net LED401_VCC: LED401.A, R404.2
- new net ANY_INPUT: A200.9, J400.4, U1106.1
- net !NO: now also J400.5; no longer J400.3
- net GND: no longer S402.2
- net INPUT_0: now also J400.7; no longer J400.5
- net INPUT_1: now also J400.9; no longer J400.7
- net INPUT_2: now also J400.11; no longer J400.9
- net INPUT_3: now also J400.13; no longer J400.11
- net INPUT_4: now also J400.8; no longer J400.6
- net INPUT_5: now also J400.10; no longer J400.8
- net INPUT_6: now also J400.12; no longer J400.10
- net INPUT_7: now also J400.14; no longer J400.12
- net INPUT_LOCK_EXT: now also J400.3, R404.1; no longer LED401.C, S402.C
- net NO_RESET_PULSE: now also J400.6; no longer J400.4
- net VCC: now also R404.2; no longer R404.1, S402.1
Routing:
- net ANY_INPUT: track 0.00 -> 385.7 mm, vias 0 -> 3
- net INPUT_0: track 203.4 -> 212.4 mm
- net INPUT_1: track 197.7 -> 206.7 mm
- net INPUT_2: track 193.9 -> 202.9 mm
- net INPUT_3: track 189.1 -> 198.0 mm
- net INPUT_LOCK_EXT: track 133.2 -> 141.2 mm
- net VCC: track 2833.8 -> 2827.5 mm
- net INPUT_4: track 155.8 -> 161.4 mm
- net NO_RESET_PULSE: track 179.3 -> 184.9 mm
- net INPUT_5: track 154.8 -> 160.3 mm
- net INPUT_6: track 155.8 -> 161.2 mm
- net INPUT_7: track 157.6 -> 160.8 mm
- net GND: track 3707.2 -> 3709.8 mm
- net !NO: track 686.6 -> 684.0 mm
- net LED401_VCC: track 2.06 -> 0.00 mm
Other:
- board size 314.5 x 159.5 mm -> 314.5 x 159.8 mm
- board text added: "A<B"
- board text added: "A=B"
- board text added: "A>B"
- board text added: "CARRY"
- board text added: "MAIN BUS"
- board text added: "Output Mode"
- board text added: "RAM/INPUT ARDUINO"
- board text removed: "RAM MANUAL ARDUINO"
