File: main.brd (EAGLE design)
At the start: 314.5 x 159.8 mm, 480 parts, among them J100 DCJ0202, J400 90152-14, Q200 NMOS, Q201 PMOS, Q300 PMOS, Q400 PMOS, Q401 NMOS, Q402 NMOS, U100 NE555N, U1000 74LS173N, U1001 74LS173N, U1002 74LS245N, U1003 74LS173N, U1004 74LS173N, U1005 74LS245N, U101 NE555N, U102 NE555N, U103 74LS04N, U104 74LS08N, U105 74LS32N, U1100 74LS173N, U1101 74LS173N, U1102 74LS161N, U1106 74HCT154DW, U1107 74HCT154DW, U1108 74LS04N, U200 HM62256, U201 74LS173N, U202 74LS173N, U203 74LS173N, U204 74LS173N, U205 74LS157N, U206 74LS157N, U207 74LS157N, U208 74LS157N, U209 74HCT595D, U210 74HCT595D, U211 74HCT595D, U212 74LS245N, U213 74LS245N, U214 74LS00N, U215 74LS173N, U216 74LS173N, U217 74LS173N, U218 74LS173N, U219 74LS245N, U220 74LS245N, U300 74LS299N, U301 74LS245N, U302 74LS08N, U303 74LS00N, U304 74LS245N, U400 74LS00N, U401 74LS245N, U500 74LS161N, U501 74LS161N, U502 74LS161N, U503 74LS161N, U504 74LS245N, U505 74LS245N, U600 74LS173N, U601 74LS173N, U602 74LS173N, U603 74LS173N, U604 74LS245N, U700 74LS283N, U701 74LS283N, U702 74LS245N, U703 74LS86N, U704 74LS86N, U705 74LS85N, U706 74LS85N, U707 74LS173N, U708 74LS125N, U709 74LS153N, U800 74LS04N, U801 74LS04N, U802 74LS08N, U803 74LS08N, U804 74LS32N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

Commit message: Final design with gerber files.
Routing:
- net MAINBUS_3: track 978.3 -> 979.1 mm
- net GND: track 3709.8 -> 3710.5 mm
- net MEM_!WE!_MAN: track 120.3 -> 120.8 mm
- added copper zone on layer 1, net LOGO
Other:
- board text added: "8 Bit Computer"
- board text added: "AI"
- board text added: "AO"
- board text added: "BI"
- board text added: "CE"
- board text added: "CI"
- board text added: "CMP"
- board text added: "CMPO"
- board text added: "CO"
- board text added: "CPB0"
- board text added: "CPB1"
- board text added: "CPTC"
- board text added: "DC 5V"
- board text added: "EO"
- board text added: "FE"
- board text added: "FI"
- board text added: "FO"
- board text added: "HLT"
- board text added: "II"
- board text added: "Input Index"
- board text added: "Instruction"
- board text added: "JLCJLCJLCJLC"
- board text added: "MHI"
- board text added: "MLI"
- board text added: "Micro- instruction"
- board text added: "NO"
- board text added: "OI"
- board text added: "OMI"
- board text added: "OO"
- board text added: "Output Index"
- board text added: "PI"
- board text added: "PO"
- board text added: "RI"
- board text added: "RM"
- board text added: "RMSB"
- board text added: "RO"
- board text added: "SM0"
- board text added: "SM1"
- board text added: "SO"
- board text added: "SRO"
- board text added: "SUB"
- board text added: "T0"
- board text added: "T1"
- board text added: "TO"
- board text added: "VI"
- board text added: "VO"
- board text added: "XI"
- board text added: "XR"
- board text added: "ZHI"
- board text added: "ZHO"
- board text added: "ZLI"
- board text added: "ZLO"
- board text added: "©2019 BlockWorker blockworker.de"

Commit message: Fixed issues encountered during build and testing.
Parts:
- added C1109, C1110: 0.1µF, rcl:C0805K
- added C403: 10nF, rcl:C0805K
- added Q403: NMOS, ExtraParts:SOT23
- added R405: 1kΩ, resistor:R0805
- R100, R101: value 330Ω -> 150Ω
- moved C1107 7.50 mm to (285.8, 49.0)
- moved RN300 1.27 mm to (32.5, 46.1)
Connections:
- new net ARDUINO_DETECT_GND: A200.14, Q200.1, R200.1, U209.13, U210.13, U211.13
- new net MEM_!OE_INT: U103.8, U105.1
- new net NO_RESET: A200.25, C403.1, J400.6, R405.1, S401.3, S401.4
- net GND: now also C1109.2, C1110.2, Q403.2; no longer A200.14, Q200.1, R200.1, U209.13, U210.13, U211.13
- net LCD_VDD: now also Q403.3
- net MEM_!OE: now also U105.3; no longer U103.8
- net NO_RESET_PULSE: now also C403.2; no longer A200.25, J400.6, S401.3, S401.4
- net RI: now also U105.2
- net RM: now also C1109.1
- net RMSB: now also C1110.1
- net RST: now also Q403.1
- net VCC: now also R405.2
Routing:
- net NO_RESET: track 0.00 -> 179.5 mm, vias 0 -> 2
- net NO_RESET_PULSE: track 184.9 -> 6.18 mm, vias 2 -> 0
- net ARDUINO_DETECT_GND: track 0.00 -> 75.4 mm, vias 0 -> 6
- net MEM_!OE_INT: track 0.00 -> 57.8 mm, vias 0 -> 3
- net RI: track 213.0 -> 230.3 mm, vias 2 -> 3
- net RST: track 691.1 -> 705.0 mm, vias 15 -> 16
- net LCD_VDD: track 2.69 -> 11.2 mm
- net MEM_!OE: track 38.6 -> 47.1 mm, vias 1 -> 2
- net GND: track 3710.5 -> 3716.6 mm, vias 57 -> 59
- net VCC: track 2827.9 -> 2830.7 mm, vias 47 -> 48
- net RM: track 369.0 -> 371.7 mm
- net RO: track 185.9 -> 183.4 mm
- net INPUT_3: track 198.0 -> 195.7 mm
- net RMSB: track 378.5 -> 379.8 mm
- net MAINBUS_3: track 979.1 -> 980.1 mm
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
Commit message: Moved library over to central BW lib, added gitignore
Parts:
- A200: device 8BitCpuParts:ARDUINO_NANO_V3 -> BW-Active:ARDUINO_NANO_V3
- DS400: device 8BitCpuParts:HD44780_LCD -> BW-Active:HD44780_LCD
- DS900, DS901, DS902, DS903: device 8BitCpuParts:LED_7SEG -> BW-Active:LED_7SEG
- J400: device 8BitCpuParts:90152-14 -> BW-Connectors:90152-14
- Q200, Q201, Q300, Q400, Q401, Q402, Q403: device ExtraParts:SOT23 -> BW-Active:SOT23
- RN1000, RN1001, RN1100, RN1101, RN1102, RN1103, RN1104, RN1105, RN1106, RN1107, RN200, RN201, RN202, RN203, RN204, RN205, RN206, RN207, RN300, RN301, RN302, RN400, RN500, RN501, RN600, RN601, RN700, RN800, RN900: device 8BitCpuParts:CAY16102J8LF -> BW-PassiveMechanical:CAY16102J8LF
- S100, S204, S300, S401: device ExtraParts:TL3305_MICROSWITCH -> BW-PassiveMechanical:TL3305_MICROSWITCH
- S101, S200: device 8BitCpuParts:ESP10 -> BW-PassiveMechanical:ESP10
- S201, S202, S203, S400: device 8BitCpuParts:DS-08 -> BW-PassiveMechanical:DIPSW-08
- U1102, U500, U501, U502, U503, U901: device 8BitCpuParts:DIL16 -> BW-Active:DIL16
